File: Hardware/Ricardo-Garnet.kicad_pcb (KiCad board)
At the start: 4 copper layers, 38.5 x 65 mm, 127 parts, among them K1 SERVO, P1 HALL/Encoder, P101 CANBUS, P2 SWD, P3 PWR_COMM, P4 IN+, P5 IN-, P6 MOTOR1, P7 MOTOR2, P9 MOTOR3, Q1 IRFS7530, Q2 IRFS7530, Q3 IRFS7530, Q4 IRFS7530, Q5 IRFS7530, Q6 IRFS7530, U1 STM32F40X_LQFP64, U2 TC2117, U3 DRV8302, U401 SN65HVD232, X1 MINI-USB-SHIELD-32005-201, X2 8MHz 10ppm

Commit message: chatting to fang
Parts:
- removed 1PIN (x2): P***, 1pin
- removed 1PIN (x2): P***, Connect:1pin
- removed C24, C401: 2.2u, CRF1:SMD-0603_c
- removed C25: 100u, w_smd_cap:c_tant_B
- removed D1: GREEN, LEDs:LED-0603
- removed D2: RED, LEDs:LED-0603
- removed D3: LED, LEDs:LED-0603
- removed G***: oshw_silkscreen-back_3mm, oshw_silkscreen-back_3mm
- removed K1: SERVO, CRF1:pinhead-1X03
- removed P1: HALL/Encoder, CRF1:MICRO_JST_6
- removed P101: CANBUS, JST conn:b4b-ph-kl
- removed P2: SWD, CRF1:MICRO_JST_6
- removed P3: PWR_COMM, CRF1:b7b-ph-kl
- removed R103, R104: 22R, CRF1:SMD-0603_r
- removed R12, R13, R22: 2k2, CRF1:SMD-0603_r
- removed R37, R38: 100R, CRF1:SMD-0603_r
- removed R401: NI, CRF1:SMD-0603_r
- removed R402: 10k, CRF1:SMD-0603_r
- removed U2: TC2117, CRF1:SOT-223
- removed U401: SN65HVD232, CRF1:SOIC-8-W
- removed X1: MINI-USB-SHIELD-32005-201, CRF1:USB-UX60R-MB-5ST
- removed X2: 8MHz 10ppm, CRF1:Crystal_5x3mm
- added 12VLED1: RED_LED, Resistor_SMD:R_0402_1005Metric, F.Cu at (158.3, 101.9)
- added 3V3LED1: BLUE_LED, Resistor_SMD:R_0402_1005Metric, F.Cu at (158.3, 103.9)
- added C100: 0.1uF, Capacitor_SMD:C_0402_1005Metric, F.Cu at (153.3, 114.1)
- added C101: 0.1uF, Capacitor_SMD:C_0402_1005Metric, F.Cu at (153.3, 116.0)
- added C42: 10uF, Capacitor_SMD:C_0402_1005Metric, F.Cu at (80.4, 124.6)
- added C45: 4.7uF, Capacitor_SMD:C_0402_1005Metric, F.Cu at (80.4, 126.8)
- added C46: 10uF, Capacitor_SMD:C_0402_1005Metric, F.Cu at (88.8, 127.7)
- added C47: 0.1uF, Capacitor_SMD:C_0402_1005Metric, F.Cu at (89.8, 127.7)
- added C48: 47uF, Capacitor_SMD:C_1206_3216Metric, F.Cu at (142.4, 65.2)
- added C61: 100nF, Capacitor_SMD:C_0402_1005Metric, F.Cu at (100.7, 141.1)
- added C62: 10uF, Capacitor_SMD:C_0402_1005Metric, F.Cu at (102.6, 141.1)
- added C63: 47nF, Capacitor_SMD:C_0402_1005Metric, F.Cu at (97.7, 149.8)
- added C66: 1uF, Capacitor_SMD:C_0402_1005Metric, F.Cu at (134.2, 58.5)
- added C67: 4.7uF, Capacitor_SMD:C_0603_1608Metric, F.Cu at (137.6, 64.8)
- added C68: 75pF, Capacitor_SMD:C_0402_1005Metric, F.Cu at (134.2, 60.5)
- added C69: 1.8nF, Capacitor_SMD:C_0402_1005Metric, F.Cu at (134.2, 62.5)
- added C70: 10uF, Capacitor_SMD:C_0805_2012Metric, F.Cu at (137.8, 59.1)
- added C71: 2.2uF, Capacitor_SMD:C_0402_1005Metric, F.Cu at (134.2, 64.5)
- added C72: 10uF, Capacitor_SMD:C_0805_2012Metric, F.Cu at (137.8, 62.1)
- added C73: 100nF, Capacitor_SMD:C_0402_1005Metric, F.Cu at (134.2, 66.4)
- added C74: 100nF, Capacitor_SMD:C_0402_1005Metric, F.Cu at (134.2, 68.4)
- added C75: 10uF, Capacitor_SMD:C_0603_1608Metric, F.Cu at (137.6, 67.3)
- added C76: 100nF, Capacitor_SMD:C_0402_1005Metric, F.Cu at (134.2, 70.4)
- added C77: 1uF, Capacitor_SMD:C_0402_1005Metric, F.Cu at (147.5, 108.2)
- added C78: 1uF, Capacitor_SMD:C_0402_1005Metric, F.Cu at (147.5, 110.1)
- added C79: 220nF, Capacitor_SMD:C_0402_1005Metric, F.Cu at (147.5, 112.1)
- added C80: 0.1uF, Capacitor_SMD:C_0402_1005Metric, F.Cu at (147.5, 114.1)
- added C81: 10nF, Capacitor_SMD:C_0402_1005Metric, F.Cu at (147.5, 116.0)
- added C82: 10nF, Capacitor_SMD:C_0402_1005Metric, F.Cu at (147.5, 118.0)
- added C83: 0.1uF, Capacitor_SMD:C_0402_1005Metric, F.Cu at (150.4, 108.2)
- added C92: 0.01uF, Capacitor_SMD:C_0402_1005Metric, F.Cu at (150.4, 110.1)
- added C93: 0.1uF, Capacitor_SMD:C_0402_1005Metric, F.Cu at (150.4, 112.1)
- added C94: 0.01uF, Capacitor_SMD:C_0402_1005Metric, F.Cu at (150.4, 114.1)
- added C95: 0.01uF, Capacitor_SMD:C_0402_1005Metric, F.Cu at (150.4, 116.0)
- added C96: 0.1uF, Capacitor_SMD:C_0402_1005Metric, F.Cu at (150.4, 118.0)
- added C97: 0.01uF, Capacitor_SMD:C_0402_1005Metric, F.Cu at (153.3, 108.2)
- added C98: 0.1uF, Capacitor_SMD:C_0402_1005Metric, F.Cu at (153.3, 110.1)
- added C99: 0.1uF, Capacitor_SMD:C_0402_1005Metric, F.Cu at (153.3, 112.1)
- added CANRXLED1: CANRXLED, LED_SMD:LED_0402_1005Metric, F.Cu at (171.3, 104.6)
- added CANTXLED1: CANTXLED, LED_SMD:LED_0402_1005Metric, F.Cu at (171.3, 106.6)
- added D6: SP0503BAHT, Package_TO_SOT_SMD:SOT-143, F.Cu at (107.6, 136.5)
- added D7: SM712_SOT23, Package_TO_SOT_SMD:SOT-23, F.Cu at (103.7, 152.3)
- added IC3: AP2205-W5-7, iclr:SOT95P282X145-5N, F.Cu at (142.7, 59.9)
- added IC4: TPS61089RNRR, iclr:IC_TPS61089RNRR, F.Cu at (142.3, 69.0)
- added IC5: ADS131M04IRUKR, iclr:QFN40P300X300X80-21N-D, F.Cu at (186.8, 61.1)
- added J1: RBUS, iclr:Molex_Mini-Fit_Jr_5569-06A2_2x03_P4.20mm_Horizontal, F.Cu at (113.5, 146.4)
- added J2: USB_C_Receptacle_USB2.0, iclr:USB_C_Receptacle_Palconn_UTC16-G, F.Cu at (112.8, 136.7)
- added J3: Rotary Pot, iclr:Molex_Nano-Fit_105313-xx03_1x03_P2.50mm_Horizontal, F.Cu at (179.8, 50.7)
- added J4: Conn_01x02_Male, Connector_Molex:Molex_Nano-Fit_105313-xx02_1x02_P2.50mm_Horizontal, F.Cu at (134.7, 96.5)
- added J5: Conn_01x02_Male, Connector_Molex:Molex_Nano-Fit_105313-xx02_1x02_P2.50mm_Horizontal, F.Cu at (203.0, 101.9)
- added J7: Conn_01x02_Male, Connector_Molex:Molex_Nano-Fit_105313-xx02_1x02_P2.50mm_Horizontal, F.Cu at (134.7, 112.5)
- added J8: Conn_01x02_Male, Connector_Molex:Molex_Nano-Fit_105313-xx02_1x02_P2.50mm_Horizontal, F.Cu at (134.7, 120.5)
- added J9: Conn_01x02_Male, Connector_Molex:Molex_Nano-Fit_105313-xx02_1x02_P2.50mm_Horizontal, F.Cu at (134.7, 128.5)
- added JP1: Conn_01x02_Male, Connector_PinHeader_2.54mm:PinHeader_1x02_P2.54mm_Vertical, F.Cu at (115.1, 121.8)
- added JP4: TermJP, iclr:SmallerSolderJP, F.Cu at (97.9, 147.9)
- added JP5: Conn_01x02_Male, Connector_PinHeader_2.54mm:PinHeader_1x02_P2.54mm_Vertical, F.Cu at (115.1, 125.4)
- added L3: 1uH, Inductor_SMD:L_0805_2012Metric, F.Cu at (87.2, 131.8)
- added L4: 2.0nH, Inductor_SMD:L_0402_1005Metric, F.Cu at (98.4, 132.5)
- added L5: 20nH, Inductor_SMD:L_0402_1005Metric, F.Cu at (99.2, 127.9)
- added L6: SRR6038-3R3Y, iclr:IND_SRP6540-390M, F.Cu at (137.2, 53.5)
- added LED6: WHITE_LED, LED_SMD:LED_0402_1005Metric, F.Cu at (90.7, 133.8)
- added R14: 10k, Resistor_SMD:R_0402_1005Metric, F.Cu at (85.7, 136.0)
- added R15: 14k, Resistor_SMD:R_0402_1005Metric, F.Cu at (81.3, 131.9)
- added R16: 56k, Resistor_SMD:R_0402_1005Metric, F.Cu at (88.8, 125.8)
- added R31: 5.1k, Resistor_SMD:R_0402_1005Metric, F.Cu at (111.0, 142.4)
- added R39: 5.1k, Resistor_SMD:R_0402_1005Metric, F.Cu at (112.9, 142.4)
- added R40: 5.1k, Resistor_SMD:R_0402_1005Metric, F.Cu at (88.5, 133.4)
- added R41: 0, Resistor_SMD:R_0603_1608Metric, F.Cu at (104.9, 147.6)
- added R44: 60, Resistor_SMD:R_0603_1608Metric, F.Cu at (102.9, 149.8)
- added R45: 60, Resistor_SMD:R_0603_1608Metric, F.Cu at (99.9, 149.8)
- added R55: 1k, Resistor_SMD:R_0402_1005Metric, F.Cu at (164.1, 101.9)
- added R56: 1k, Resistor_SMD:R_0402_1005Metric, F.Cu at (164.1, 103.9)
- added R57: 28.7k, Resistor_SMD:R_0402_1005Metric, F.Cu at (131.3, 50.5)
- added R58: 866k, Resistor_SMD:R_0402_1005Metric, F.Cu at (131.3, 52.5)
- added R59: 92k, Resistor_SMD:R_0402_1005Metric, F.Cu at (131.3, 54.5)
- added R60: 49.9k, Resistor_SMD:R_0402_1005Metric, F.Cu at (131.3, 56.5)
- added R61: 10K, Resistor_SMD:R_0402_1005Metric, F.Cu at (131.3, 58.5)
- added R62: 332k, Resistor_SMD:R_0402_1005Metric, F.Cu at (131.3, 60.5)
- added R63: 280k, Resistor_SMD:R_0402_1005Metric, F.Cu at (131.3, 62.4)
- added R64: 8.56k, Resistor_SMD:R_0402_1005Metric, F.Cu at (147.6, 120.0)
- added R65: 432k, Resistor_SMD:R_0402_1005Metric, F.Cu at (131.3, 64.4)
- added R66: 120, Resistor_SMD:R_0402_1005Metric, F.Cu at (147.6, 122.0)
- added R67: 59, Resistor_SMD:R_0402_1005Metric, F.Cu at (147.6, 124.0)
- added R68: 1k, Resistor_SMD:R_0402_1005Metric, F.Cu at (147.6, 126.0)
- added R69: 1k, Resistor_SMD:R_0402_1005Metric, F.Cu at (150.5, 120.0)
- added R72: 1k, Resistor_SMD:R_0402_1005Metric, F.Cu at (150.5, 122.0)
- added R73: 100, Resistor_SMD:R_0402_1005Metric, F.Cu at (150.5, 124.0)
- added R74: 59, Resistor_SMD:R_0402_1005Metric, F.Cu at (150.5, 126.0)
- added R75: 100, Resistor_SMD:R_0402_1005Metric, F.Cu at (153.4, 120.0)
- added R76: 1k, Resistor_SMD:R_0402_1005Metric, F.Cu at (153.4, 122.0)
- added R80: 100, Resistor_SMD:R_0402_1005Metric, F.Cu at (153.4, 124.0)
- added R81: 100, Resistor_SMD:R_0402_1005Metric, F.Cu at (153.4, 126.0)
- added TP1: TestPoint, TestPoint:TestPoint_Pad_D1.0mm, F.Cu at (119.8, 138.0)
- added TP10: TestPoint, TestPoint:TestPoint_Pad_D1.0mm, F.Cu at (109.2, 124.2)
- added TP2: TestPoint, TestPoint:TestPoint_Pad_D1.0mm, F.Cu at (120.6, 134.5)
- added TP5: TestPoint, TestPoint:TestPoint_Pad_D1.5mm, F.Cu at (86.0, 137.8)
- added TP6: TestPoint, TestPoint:TestPoint_Pad_D1.5mm, F.Cu at (89.4, 131.2)
- added TP9: TestPoint, TestPoint:TestPoint_Pad_D1.0mm, F.Cu at (111.3, 124.3)
- added TXLED1: GREEN_LED, Resistor_SMD:R_0402_1005Metric, F.Cu at (110.8, 126.3)
- added U10: MAX31856, Package_SO:TSSOP-14_4.4x5mm_P0.65mm, F.Cu at (186.0, 114.8)
- added U11: MAX31856, Package_SO:TSSOP-14_4.4x5mm_P0.65mm, F.Cu at (186.6, 121.8)
- added U4: LM66200DRLR, iclr:SOTFL50P160X60-8N, F.Cu at (83.5, 136.9)
- added U5: SC4215, iclr:SOIC127P599X175-9N, F.Cu at (84.6, 125.7)
- added U6: SN65HVD230, Package_SO:SOIC-8_3.9x4.9mm_P1.27mm, F.Cu at (101.4, 145.3)
- added U7: MAX77827AEFD+T, iclr:CONV_MAX77827AEFD+T, F.Cu at (83.5, 131.8)
- added U9: THVD2429, iclr:TPS74901DRCR, F.Cu at (191.2, 106.4)
- added Y2: R940000171, iclr:Crystal_SMD_2016-4Pin_2.0x1.6mm, F.Cu at (98.2, 125.7)
- C1, C39, C40, C43, C44, C49, C8, C9: footprint CRF1:SMD-1206 -> Capacitor_SMD:C_1206_3216Metric
- C10, C35: value 2.2u -> 1uF; footprint CRF1:SMD-0603_c -> Capacitor_SMD:C_0402_1005Metric
- C11, C13: value 2.2u -> 0.1uF; footprint CRF1:SMD-0603_c -> Capacitor_SMD:C_0402_1005Metric
- C12: value 2.2u -> 10nF; footprint CRF1:SMD-0603_c -> Capacitor_SMD:C_0402_1005Metric
- C14: value 2.2u -> 1uF; footprint CRF1:SMD-0603_c -> Capacitor_SMD:C_0402_1005Metric; moved to F.Cu
- C15: value 15p -> 0.1uF; footprint CRF1:SMD-0603_c -> Capacitor_SMD:C_0402_1005Metric; moved to F.Cu
- C16: value 2.2u -> 0.1uF; footprint CRF1:SMD-0603_c -> Capacitor_SMD:C_0402_1005Metric; moved to F.Cu
- C17, C31: value 2.2u -> 11pF; footprint CRF1:SMD-0603_c -> Capacitor_SMD:C_0402_1005Metric; moved to F.Cu
- C18, C19, C20, C21, C22, C23, C26, C27, C28, C29, C30, C34, C36, C41, C52: footprint CRF1:SMD-0603_c -> Capacitor_SMD:C_0603_1608Metric
- C2: footprint CRF1:SMD-0603_c -> Capacitor_SMD:C_0603_1608Metric; moved to F.Cu
- C3: value 100n -> 10uF; footprint CRF1:SMD-0603_c -> Capacitor_SMD:C_0402_1005Metric; moved to F.Cu
- C32: value 100n -> 10uF; footprint CRF1:SMD-0603_c -> Capacitor_SMD:C_0603_1608Metric; moved to F.Cu
- C37, C51: footprint w_smd_cap:c_2220 -> Capacitor_SMD:C_2220_5750Metric
- C38: value 15p -> 22uF; footprint CRF1:SMD-0603_c -> Capacitor_SMD:C_0603_1608Metric; moved to F.Cu
- C4, C5: value 4n7 -> 0.1uF; footprint CRF1:SMD-0603_c -> Capacitor_SMD:C_0402_1005Metric; moved to F.Cu
- C6: value 4n7 -> 1uF; footprint CRF1:SMD-0603_c -> Capacitor_SMD:C_0402_1005Metric; moved to F.Cu
- C7: value 4n7 -> 10uF; footprint CRF1:SMD-0603_c -> Capacitor_SMD:C_0402_1005Metric; moved to F.Cu
- D5: moved to F.Cu
- R1, R25, R28, R29, R30, R34, R35, R36, R42, R43, R46, R48, R49, R50, R51: footprint CRF1:SMD-0603_r -> Resistor_SMD:R_0603_1608Metric
- R10: value 10k -> 3k; footprint CRF1:SMD-0603_r -> Resistor_SMD:R_0402_1005Metric; moved to F.Cu
- R11: value 2k2 -> 10k; footprint CRF1:SMD-0603_r -> Resistor_SMD:R_0402_1005Metric; moved to F.Cu
- R17, R18, R19, R2: footprint CRF1:SMD-0603_r -> Resistor_SMD:R_0402_1005Metric
- R20: footprint CRF1:SMD-0603_r -> Resistor_SMD:R_0402_1005Metric; moved to B.Cu
- R21, R24, R27, R33, R4: footprint CRF1:SMD-0603_r -> Resistor_SMD:R_0402_1005Metric; moved to F.Cu
- R23, R26, R3, R32: footprint CRF1:SMD-0603_r -> Resistor_SMD:R_0603_1608Metric; moved to F.Cu
- R5: value 2k2 -> 470; footprint CRF1:SMD-0603_r -> Resistor_SMD:R_0402_1005Metric; moved to F.Cu
- R6: value 0R -> 499R; footprint CRF1:SMD-0603_r -> Resistor_SMD:R_0402_1005Metric; moved to F.Cu
- R7, R8: value 10k -> 10K; footprint CRF1:SMD-0603_r -> Resistor_SMD:R_0402_1005Metric; moved to F.Cu
- R9: value 10k -> 470; footprint CRF1:SMD-0603_r -> Resistor_SMD:R_0402_1005Metric; moved to F.Cu
- U1: value STM32F40X_LQFP64 -> ESP32-S3; footprint CRF1:lqfp64_pad_mod -> iclr:QFN40P700X700X90-57N
- moved C13 82.4 mm to (170.3, 98.7), turned to 0 degrees
- moved R9 76.6 mm to (161.2, 107.9), turned to 0 degrees
- moved C12 76.3 mm to (170.3, 96.7), turned to 0 degrees
- moved R10 73.0 mm to (161.2, 109.8), turned to 0 degrees
- moved C11 70.3 mm to (170.3, 94.7), turned to 0 degrees
- moved C10 63.6 mm to (167.5, 102.6), turned to 0 degrees
- moved C41 58.5 mm to (167.8, 109.9), turned to 0 degrees
- moved R1 52.8 mm to (167.8, 104.9)
- moved R21 35.4 mm to (127.5, 109.7)
- moved R4 35.3 mm to (114.8, 109.7), turned to -90 degrees
- moved C2 35.1 mm to (113.6, 109.4)
- moved D5 32.5 mm to (129.0, 106.5), turned to 0 degrees
- moved R7 31.8 mm to (112.8, 122.5)
- moved R6 31.7 mm to (111.8, 126.3), turned to -90 degrees
- moved R3 31.5 mm to (113.6, 112.4), turned to 90 degrees
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Connections:
- net /MCU/H3 renamed /H3
- C10 pad 1: GND -> VCC
- C10 pad 2: VCC -> GND
- C11 pad 1: GND -> VCC
- C11 pad 2: VCC -> GND
- C12 pad 1: GND -> VCC
- C12 pad 2: VCC -> GND
- C13 pad 1: GND -> VCC
- C13 pad 2: VCC -> GND
- C14 pad 1: GND -> /CHIP_PU
- C14 pad 2: VCC -> GND
- C15 pad 1: Net-(C15-Pad1) -> /CHIP_PU
- C16 pad 1: Net-(C16-Pad1) -> /BOOT
- C18 pad 1: Net-(C18-Pad1) -> GND
- C18 pad 2: GND -> Net-(U3-GVDD)
- C2 pad 2: /MCU/AN_IN -> /AN_IN
- C26 pad 1: Net-(C18-Pad1) -> GND
- C26 pad 2: GND -> Net-(U3-GVDD)
- C3 pad 1: GND -> /Power/BBIN
- C3 pad 2: /MCU/SERVO -> GND
- C31 pad 1: GND -> Net-(U1-XTAL_N)
- C31 pad 2: VCC -> GND
- C32 pad 1: GND -> /Power/BBIN
- C32 pad 2: NRST -> GND
- C35 pad 1: GND -> /Power/BIAS
- C35 pad 2: VCC -> GND
- C38 pad 1: Net-(C38-Pad1) -> /Power/BBOUT
- C4 pad 1: GND -> Net-(C4-Pad1)
- C4 pad 2: /Filters/TEMP_IN -> GND
- C41 pad 1: /MCU/ADC_TEMP -> /MOS_TEMP
- C5 pad 1: /Filters/HALL3_OUT -> VCC
- C6 pad 1: /Filters/HALL2_OUT -> VCC
- C7 pad 1: /Filters/HALL1_OUT -> VCC
- Q2 pad S: /Mosfet driver/H1_LOW -> GND
- Q6 pad S: /Mosfet driver/H3_LOW -> GND
- R1 pad 2: /MCU/ADC_TEMP -> /MOS_TEMP
- R10 pad 1: /Filters/HALL3_IN -> DEP
- R10 pad 2: /Filters/HALL3_OUT -> Net-(12VLED1-A)
- R11 pad 1: /Filters/HALL3_IN -> /Power/FBIn
- R11 pad 2: VCC -> GND
- R2 pad 1: /MCU/ADC_TEMP -> /MOS_TEMP
- R23 pad 2: /MCU/SENS1 -> /SENS1
- R24 pad 2: /MCU/SENS1 -> /SENS1
- R26 pad 2: /MCU/SENS2 -> /SENS2
- R27 pad 2: /MCU/SENS2 -> /SENS2
- R3 pad 2: /MCU/AN_IN -> /AN_IN
- R30 pad 1: /Mosfet driver/H1_LOW -> GND
- R32 pad 2: /MCU/SENS3 -> /SENS3
- R33 pad 2: /MCU/SENS3 -> /SENS3
- R36 pad 1: /Mosfet driver/H1_LOW -> GND
- R4 pad 2: /MCU/AN_IN -> /AN_IN
- R46 pad 1: /Mosfet driver/H3_LOW -> GND
- R5 pad 1: /MCU/SERVO -> VCC
- R53 pad 2: /Mosfet driver/H1_LOW -> GND
- R54 pad 1: /Mosfet driver/H3_LOW -> GND
- R6 pad 1: Net-(R6-Pad1) -> /TXD
- R6 pad 2: +5V -> Net-(U1-U0TXD/PROG/GPIO43)
- R7 pad 1: /Filters/TEMP_IN -> VCC
- R7 pad 2: VCC -> /CHIP_PU
- R8 pad 1: /Filters/HALL1_IN -> VCC
- R8 pad 2: /Filters/HALL1_OUT -> /BOOT
- R9 pad 1: /Filters/HALL2_IN -> Net-(3V3LED1-A)
- R9 pad 2: /Filters/HALL2_OUT -> VCC
- U1 pad 1: VCC -> unconnected-(U1-LNA_IN/RF-Pad1)
- U1 pad 10: /MCU/AN_IN -> /BR_SO2
- U1 pad 11: Net-(U1-Pad11) -> /BR_SO1
- U1 pad 12: GND -> /AN_IN
- U1 pad 13: VCC -> /MOS_TEMP
- U1 pad 14: /MCU/SENS3 -> /HSPI_MISO
- U1 pad 15: /MCU/SENS2 -> /HSPI_MOSI
- U1 pad 16: /MCU/SENS1 -> /HSPI_SCLK
- U1 pad 17: /MCU/ADC_TEMP -> /ACD_CLK
- U1 pad 18: GND -> /MOD_RX
- U1 pad 19: VCC -> /MOD_TX
- U1 pad 2: Net-(U1-Pad2) -> Net-(C4-Pad1)
- U1 pad 20: /MCU/TX_SDA_NSS -> VCC
- U1 pad 21: /MCU/SCK_ADC_EXT -> /TC_CS_0
- U1 pad 22: /MCU/MISO_ADC_EXT2 -> /TC_CS_1
- U1 pad 23: /MCU/RX_SCL_MOSI -> /CAN_RX
- U1 pad 24: /MCU/LED_GREEN -> /CAN_TX
- U1 pad 25: /MCU/LED_RED -> /Data-
- U1 pad 26: /MCU/BR_SO2 -> /Data+
- U1 pad 27: /MCU/BR_SO1 -> /MOD_DE
- U1 pad 28: Net-(U1-Pad28) -> unconnected-(U1-SPI_CS1/GPIO26-Pad28)
- U1 pad 29: /MCU/RX_SCL_MOSI -> unconnected-(U1-VDD_SPI-Pad29)
- U1 pad 3: Net-(U1-Pad3) -> Net-(C4-Pad1)
- U1 pad 30: /MCU/TX_SDA_NSS -> unconnected-(U1-SPIHD/GPIO27-Pad30)
- U1 pad 31: Net-(C16-Pad1) -> unconnected-(U1-SPIWP/GPIO28-Pad31)
- U1 pad 32: VCC -> unconnected-(U1-SPICS0/GPIO29-Pad32)
- U1 pad 33: /MCU/DC_CAL -> unconnected-(U1-SPICLK/GPIO30-Pad33)
- U1 pad 34: /MCU/L3 -> unconnected-(U1-SPIQ/GPIO31-Pad34)
- U1 pad 35: /MCU/L2 -> unconnected-(U1-SPID/GPIO32-Pad35)
- U1 pad 36: /MCU/L1 -> /ACD_CS
- U1 pad 37: /MCU/TX_SDA_NSS -> unconnected-(U1-SPICLK_P/GPIO47-Pad37)
- U1 pad 38: /MCU/RX_SCL_MOSI -> unconnected-(U1-GPIO33-Pad38)
- U1 pad 39: Net-(U1-Pad39) -> /EN_GATE
- U1 pad 4: Net-(U1-Pad4) -> /CHIP_PU
- U1 pad 40: Net-(U1-Pad40) -> /L3
- U1 pad 42: /MCU/H2 -> /L2
- U1 pad 43: /MCU/H1 -> /H2
- U1 pad 44: /MCU/USB_DM -> /L1
- U1 pad 45: /MCU/USB_DP -> /H1
- U1 pad 46: SWDIO -> VCC
- U1 pad 47: Net-(C17-Pad1) -> /DC_CAL
- U1 pad 48: VCC -> /FAULT
- U1 pad 49: SWCLK -> Net-(U1-U0TXD/PROG/GPIO43)
- U1 pad 5: Net-(C15-Pad1) -> /BOOT
- U1 pad 50: Net-(U1-Pad50) -> /RXD
- U1 pad 51: /MCU/EN_GATE -> unconnected-(U1-GPIO45-Pad51)
- U1 pad 52: /Filters/HALL3_OUT -> unconnected-(U1-GPIO46-Pad52)
- U1 pad 53: /MCU/FAULT -> Net-(U1-XTAL_N)
- U1 pad 55: Net-(U1-Pad55) -> VCC
- U1 pad 56: Net-(U1-Pad56) -> VCC
- U1 pad 57: /MCU/SERVO -> GND
- U1 pad 6: Net-(C38-Pad1) -> /SENS3
- U1 pad 7: NRST -> /SENS1
- U1 pad 8: /Filters/TEMP_IN -> unconnected-(U1-GPIO3/ADC1_CH2-Pad8)
- U1 pad 9: Net-(U1-Pad9) -> /SENS2
- U3 pad 12: /MCU/DC_CAL -> /DC_CAL
- U3 pad 13: Net-(C18-Pad1) -> Net-(U3-GVDD)
- U3 pad 16: /MCU/EN_GATE -> /EN_GATE
- U3 pad 17: /MCU/H1 -> /H1
- U3 pad 18: /MCU/L1 -> /L1
- U3 pad 19: /MCU/H2 -> /H2
- U3 pad 20: /MCU/L2 -> /L2
- U3 pad 22: /MCU/L3 -> /L3
- U3 pad 25: /MCU/BR_SO1 -> /BR_SO1
- U3 pad 26: /MCU/BR_SO2 -> /BR_SO2
- U3 pad 34: /Mosfet driver/H3_LOW -> GND
- U3 pad 4: Net-(U3-Pad4) -> unconnected-(U3-PWRGD-Pad4)
- U3 pad 44: /Mosfet driver/H1_LOW -> GND
- U3 pad 5: Net-(U3-Pad5) -> unconnected-(U3-OCTW-Pad5)
- U3 pad 55: Net-(U3-Pad55) -> unconnected-(U3-EN_BUCK-Pad55)
- U3 pad 56: Net-(U3-Pad56) -> unconnected-(U3-SS_TR-Pad56)
- U3 pad 6: /MCU/FAULT -> /FAULT
Routing:
- net VCC: track 185.2 -> 11.0 mm, vias 9 -> 4
- net GND: track 398.8 -> 264.0 mm, vias 27 -> 50
- net +5V: track 115.3 -> 15.1 mm, vias 4 -> 1
- net /Mosfet driver/H3_LOW: track 53.5 -> 0.00 mm, vias 2 -> 0
- net /Mosfet driver/H1_LOW: track 48.5 -> 0.00 mm, vias 2 -> 0
- net /MCU/TX_SDA_NSS: track 47.1 -> 0.00 mm, vias 2 -> 0
- net /MCU/ADC_TEMP: track 44.0 -> 0.00 mm
- net /MOS_TEMP: track 0.00 -> 41.7 mm, vias 0 -> 2
- net /MCU/RX_SCL_MOSI: track 41.6 -> 0.00 mm, vias 1 -> 0
- net /MCU/MISO_ADC_EXT2: track 36.0 -> 0.00 mm, vias 1 -> 0
- net /AN_IN: track 0.00 -> 34.1 mm, vias 0 -> 2
- net NRST: track 32.6 -> 0.00 mm, vias 2 -> 0
- net /MCU/SENS3: track 30.2 -> 0.00 mm, vias 2 -> 0
- net /MCU/AN_IN: track 28.9 -> 0.00 mm, vias 2 -> 0
- net /MCU/SENS2: track 28.6 -> 0.00 mm, vias 2 -> 0
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- added copper zone on F.Cu, net /AN_IN
- added copper zone on F.Cu, net /Power/BBIN
- added copper zone on F.Cu, net /Power/BBOUT
- added copper zone on B.Cu, net /Power/LX1
- added copper zone on F.Cu, net /Power/LX1
- added copper zone on B.Cu, net /Power/LX2
- added copper zone on F.Cu, net /Power/LX2
- added copper zone on F.Cu, net /TXD
- added copper zone on F.Cu, net VCC
- removed copper zone on B.Cu, net /Mosfet driver/H1_LOW
- removed copper zone on B.Cu, net /Mosfet driver/H3_LOW
- removed copper zone on B.Cu, net VCC
Other:
- board size 38.5 x 65 mm -> 38.5 x 80 mm
