File: Hardware/_autosave-Ricardo-Garnet.kicad_pcb (KiCad board)
At the start: 4 copper layers, 38.5 x 80 mm, 193 parts, among them IC3 AP2205-W5-7, IC4 TPS61089RNRR, IC5 ADS131M04IRUKR, J1 RBUS, J2 USB_C_Receptacle_USB2.0, J3 Rotary Pot, J4 Conn_01x02_Male, J5 Conn_01x02_Male, J7 Conn_01x02_Male, J8 Conn_01x02_Male, J9 Conn_01x02_Male, P4 IN+, P5 IN-, P6 MOTOR1, P7 MOTOR2, P9 MOTOR3, Q1 IRFS7530, Q2 IRFS7530, Q3 IRFS7530, Q4 IRFS7530, Q5 IRFS7530, Q6 IRFS7530, U1 ESP32-S3, U10 MAX31856, U11 MAX31856, U3 DRV8302, U4 LM66200DRLR, U5 SC4215, U6 SN65HVD230, U7 MAX77827AEFD+T, U9 THVD2429, Y2 R940000171

Commit message: commit pre-hackspace request
Parts:
- moved J4 65.1 mm to (81.1, 133.4), turned to 180 degrees
- moved J7 53.9 mm to (81.1, 118.0), turned to 180 degrees
- moved J8 53.9 mm to (81.1, 125.8), turned to 180 degrees
- moved TP5 8.83 mm to (102.9, 136.5)
- moved C42 7.13 mm to (88.2, 142.2)
- moved U4 7.13 mm to (100.5, 139.1)
- moved C47 7.13 mm to (91.3, 132.8)
- moved C3 7.13 mm to (98.7, 140.4)
- moved R15 7.13 mm to (95.5, 141.3)
- moved U7 7.13 mm to (95.4, 139.1)
- moved C32 7.13 mm to (97.9, 137.5)
- moved C35 7.13 mm to (97.7, 140.4)
- moved C38 7.13 mm to (92.8, 137.5)
- moved C45 7.13 mm to (90.4, 142.2)
- moved C46 7.13 mm to (91.3, 133.8)
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