File: Hardware/Ricardo-Garnet.kicad_sch (KiCad schematic)
At the start: 47 parts, among them J1 RBUS, P4 IN+, P5 IN-, U1 ESP32-S3, Y2 R940000171

Commit message: touching up and adding thermals for coating
Connections:
- net GND: no longer H2.1, H3.1
- no-connect marks 15 -> 17
Changed lines of the file:
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@@
 	)
 	(junction
-		(at 185.42 35.56)
-		(diameter 0)
-		(color 0 0 0 0)
-	)
-	(junction
 		(at 237.49 21.59)
 		(diameter 0)
@@
 	)
 	(junction
-		(at 187.96 35.56)
-		(diameter 0)
-		(color 0 0 0 0)
-	)
-	(junction
 		(at 266.7 157.48)
 		(diameter 0)
@@
 	)
 	(junction
-		(at 190.5 35.56)
-		(diameter 0)
-		(color 0 0 0 0)
-	)
-	(junction
 		(at 269.24 144.78)
 		(diameter 0)
@@
 	)
 	(no_connect
+		(at 190.5 35.56)
+	)
+	(no_connect
 		(at 133.35 101.6)
 	)
@@
 	)
 	(no_connect
+		(at 185.42 35.56)
+	)
+	(no_connect
 		(at 133.35 73.66)
 	)
@@
 	(wire
 		(pts
-			(xy 187.96 35.56) (xy 185.42 35.56)
-		)
-		(stroke
-			(width 0)
-			(type default)
-		)
-	)
-	(wire
-		(pts
 			(xy 133.35 88.9) (xy 139.7 88.9)
 		)
@@
 	(wire
 		(pts
-			(xy 195.58 35.56) (xy 190.5 35.56)
-		)
-		(stroke
-			(width 0)
-			(type default)
-		)
-	)
-	(wire
-		(pts
 			(xy 207.01 129.54) (xy 208.28 129.54)
 		)
@@
 	(wire
 		(pts
-			(xy 185.42 35.56) (xy 180.34 35.56)
-		)
-		(stroke
-			(width 0)
-			(type default)
-		)
-	)
-	(wire
-		(pts
 			(xy 237.49 143.51) (xy 246.38 143.51)
 		)
@@
 	(wire
 		(pts
-			(xy 190.5 35.56) (xy 187.96 35.56)
-		)
-		(stroke
-			(width 0)
-			(type default)
-		)
-	)
-	(wire
-		(pts
 			(xy 269.24 143.51) (xy 269.24 142.24)
 		)
@@
 	)
 	(symbol
+		(lib_name "GND-RESCUE-BLDC_4_25")
+		(lib_id "BLDC_4-rescue:GND-RESCUE-BLDC_4")
+		(at 195.58 35.56 0)
+		(unit 1)
+		(exclude_from_sim no)
+		(in_bom yes)
+		(on_board yes)
+		(dnp no)
+		(property "Reference" "#PWR058"
+			(at 195.58 35.56 0)
+			(effects
+				(font
+					(size 0.762 0.762)
+				)
+				(hide yes)
+			)
+		)
+		(property "Value" "GND"
+			(at 195.58 37.338 0)
+			(effects
+				(font
+					(size 0.762 0.762)
+				)
+				(hide yes)
+			)
+		)
+		(property "Footprint" ""
+			(at 195.58 35.56 0)
+			(effects
+				(font
+					(size 1.524 1.524)
+				)
+				(hide yes)
+			)
+		)
+		(property "Datasheet" ""
+			(at 195.58 35.56 0)
+			(effects
+				(font
+					(size 1.524 1.524)
+				)
+				(hide yes)
+			)
+		)
+		(property "Description" ""
+			(at 195.58 35.56 0)
+			(effects
+				(font
+					(size 1.27 1.27)
+				)
+			)
+		)
+		(pin "1"
+		)
+		(instances
+			(project "Ricardo-Garnet"
+				(path "/a4c716a5-e5f4-4cd7-812e-2c21e63f692f"
+					(reference "#PWR058")
+					(unit 1)
+				)
+			)
+		)
+	)
+	(symbol
 		(lib_name "GND-RESCUE-BLDC_4_20")
 		(lib_id "BLDC_4-rescue:GND-RESCUE-BLDC_4")
@@
 	)
 	(symbol
+		(lib_name "GND-RESCUE-BLDC_4_25")
+		(lib_id "BLDC_4-rescue:GND-RESCUE-BLDC_4")
+		(at 180.34 35.56 0)
+		(unit 1)
+		(exclude_from_sim no)
+		(in_bom yes)
+		(on_board yes)
+		(dnp no)
+		(property "Reference" "#PWR057"
+			(at 180.34 35.56 0)
+			(effects
+				(font
+					(size 0.762 0.762)
+				)
+				(hide yes)
+			)
+		)
+		(property "Value" "GND"
+			(at 180.34 37.338 0)
+			(effects
+				(font
+					(size 0.762 0.762)
+				)
+				(hide yes)
+			)
+		)
+		(property "Footprint" ""
+			(at 180.34 35.56 0)
+			(effects
+				(font
+					(size 1.524 1.524)
+				)
+				(hide yes)
+			)
+		)
+		(property "Datasheet" ""
+			(at 180.34 35.56 0)
+			(effects
+				(font
+					(size 1.524 1.524)
+				)
+				(hide yes)
+			)
+		)
+		(property "Description" ""
+			(at 180.34 35.56 0)
+			(effects
+				(font
+					(size 1.27 1.27)
+				)
+			)
+		)
+		(pin "1"
+		)
+		(instances
+			(project "Ricardo-Garnet"
+				(path "/a4c716a5-e5f4-4cd7-812e-2c21e63f692f"
+					(reference "#PWR057")
+					(unit 1)
+				)
+			)
+		)
+	)
+	(symbol
 		(lib_name "VCC_14")
 		(lib_id "BLDC_4-rescue:VCC")
@@
 					(unit 1)
 				)
-			)
-		)
-	)
-	(symbol
-		(lib_id "power:GND")
-		(at 187.96 35.56 0)
-		(unit 1)
-		(exclude_from_sim no)
-		(in_bom yes)
-		(on_board yes)
-		(dnp no)
-		(property "Reference" "#PWR057"
-			(at 187.96 41.91 0)
-			(effects
-				(font
-					(size 1.27 1.27)
-				)
-				(hide yes)
-			)
-		)
-		(property "Value" "GND"
-			(at 188.087 39.9542 0)
-			(effects
-				(font
-					(size 1.27 1.27)
-				)
-			)
-		)
-		(property "Footprint" ""
-			(at 187.96 35.56 0)
-			(effects
-				(font
-					(size 1.27 1.27)
-				)
-				(hide yes)
-			)
-		)
-		(property "Datasheet" ""
-			(at 187.96 35.56 0)
-			(effects
-				(font
-					(size 1.27 1.27)
-				)
-				(hide yes)
-			)
-		)
-		(property "Description" "Power symbol creates a global label with name \"GND\" , ground"
-			(at 187.96 35.56 0)
-			(effects
-				(font
-					(size 1.27 1.27)
-				)
-				(hide yes)
-			)
-		)
-		(pin "1"
-		)
-		(instances
-			(project "Ricardo-Garnet"
-				(path "/a4c716a5-e5f4-4cd7-812e-2c21e63f692f"
-					(reference "#PWR057")
-					(unit 1)
-				)

Commit message: added 2wire sensor and silkscreen
Parts:
- 12VLED1, 3V3LED1, TXLED1: footprint Resistor_SMD:R_0402_1005Metric -> LED_SMD:LED_0402_1005Metric
Connections:
- net MOD_DE renamed MOD_DIR
Other:
- sheet sensors ports: added MOD_BUS_DIR; removed MOD_BUS_DE
- company: Benjamin Vedder -> (none)
- title: BLDC Driver 4.11 -> (none)
