File: Hardware/Ricardo-Garnet.kicad_sch (KiCad schematic)
At the start: 47 parts, among them J1 RBUS, P4 IN+, P5 IN-, U1 ESP32-S3, Y2 R940000171

Commit message: changes made post will's review
Parts:
- removed C2: 100n, Capacitor_SMD:C_0603_1608Metric, symbol BLDC_4-rescue:C-RESCUE-BLDC_4
- removed C41: 2.2u, Capacitor_SMD:C_0603_1608Metric, symbol BLDC_4-rescue:C-RESCUE-BLDC_4
- removed R1: NTC 10k, Resistor_SMD:R_0603_1608Metric, symbol BLDC_4-rescue:R-RESCUE-BLDC_4
- removed R2: 10k, Resistor_SMD:R_0402_1005Metric, symbol BLDC_4-rescue:R-RESCUE-BLDC_4
- removed R3: 39k, Resistor_SMD:R_0603_1608Metric, symbol BLDC_4-rescue:R-RESCUE-BLDC_4
- removed R4: 2k2, Resistor_SMD:R_0402_1005Metric, symbol BLDC_4-rescue:R-RESCUE-BLDC_4
- added C114: 100nF, Capacitor_SMD:C_0402_1005Metric, symbol Device:C_Small
- added C115: 2.2uF, Capacitor_SMD:C_0402_1005Metric, symbol Device:C_Small
- added R109: 39kΩ, Resistor_SMD:R_0402_1005Metric, symbol Device:R_Small
- added R110: 2.2kΩ, Resistor_SMD:R_0402_1005Metric, symbol Device:R_Small
- added R111: NCU15XH103F6SRC, easyeda2kicad:R0402, symbol easyeda2kicad:NCU15XH103F6SRC
- added R112: 10kΩ, Resistor_SMD:R_0402_1005Metric, symbol Device:R_Small
- C101: renamed from C7; footprint Capacitor_SMD:C_0402_1005Metric -> Capacitor_SMD:C_0603_1608Metric
- C104: renamed from C15; value 0.1uF -> 100nF
- C105: renamed from C5; value 0.1uF -> 100nF
- C106: renamed from C4; value 0.1uF -> 100nF
- C109: renamed from C11; value 0.1uF -> 100nF
- C110: renamed from C16; value 0.1uF -> 100nF
- C111: renamed from C13; value 0.1uF -> 100nF
- CANRXLED101: renamed from CANRXLED1; value CANRXLED -> ORANGE_LED
- CANTXLED101: renamed from CANTXLED1; value CANTXLED -> GREEN_LED
- L101: renamed from L4; value 2.0nH -> 2nH
- R101: renamed from R7; value 10K -> 10kΩ
- R102: renamed from R5; value 470 -> 1kΩ
- R103: renamed from R55; value 1k -> 1kΩ
- R104: renamed from R56; value 1k -> 1kΩ
- R105: renamed from R9; value 470 -> 1kΩ
- R106: renamed from R8; value 10K -> 10kΩ
- R107: renamed from R6; value 499R -> 499Ω
- R108: renamed from R10; value 3k -> 3kΩ
- renumbered 12VLED1 to 12VLED101, 3V3LED1 to 3V3LED101, C14 to C102, C6 to C103, C10 to C107, C12 to C108, C31 to C112, C17 to C113, H1 to H101, H2 to H102, H3 to H103, H4 to H104, J1 to J101, JP1 to JP101, JP5 to JP102, L5 to L102, P4 to P101, P5 to P102, TP9 to TP101, TP10 to TP102, TXLED1 to TXLED101, U1 to U101, Y2 to Y101
Connections:
- net ACD_CLK: now also U101.11 (GPIO6/ADC1_CH5); no longer U101.12 (GPIO7/ADC1_CH6)
- net AN_IN: now also C114.2, R109.2, R110.2
- net BR_SO1: now also U101.38 (GPIO33); no longer U101.6 (GPIO1/ADC1_CH0)
- net BR_SO2: now also U101.37 (SPICLK_P/GPIO47); no longer U101.7 (GPIO2/ADC1_CH1)
- net ENCODER_CS: now also U101.36 (SPICLK_N/GPIO48); no longer U101.37 (SPICLK_P/GPIO47)
- net GND: now also C114.1, C115.2, R110.1, R112.2
- net MOD_DIR: now also U101.12 (GPIO7/ADC1_CH6); no longer U101.36 (SPICLK_N/GPIO48)
- net MOS_TEMP: now also C115.1, R111.1, R112.1
- net SENS1: now also U101.6 (GPIO1/ADC1_CH0); no longer U101.10 (GPIO5/ADC1_CH4)
- net SENS2: now also U101.7 (GPIO2/ADC1_CH1); no longer U101.11 (GPIO6/ADC1_CH5)
- net SENS3: now also U101.10 (GPIO5/ADC1_CH4); no longer U101.9 (GPIO4/ADC1_CH3)
- net V_SUPPLY: now also R109.1
- net VCC renamed +3V3
- net +3V3: now also R111.2
- new net OCTW: U101.9 (GPIO4/ADC1_CH3)
- no-connect marks 17 -> 16
Other:
- sheet Mosfet driver ports: added OCTW; removed none
- note removed: "BLDC motor controller"
- moved on the sheet: C103, C106, C107, C108, C109, C111, L101, L102, R101, R105, R106
