File: Hardware/CAN.kicad_sch (KiCad schematic)
At the start: 9 parts, among them U6 SN65HVD230

Commit message: changes made post will's review
Parts:
- C202: renamed from C62; footprint Capacitor_SMD:C_0402_1005Metric -> Capacitor_SMD:C_0603_1608Metric
- D201: renamed from D7; value SM712_SOT23 -> SM712
- R201: renamed from R41; value 0 -> 0Ω
- R202: renamed from R44; value 60 -> 60Ω
- R203: renamed from R45; value 60 -> 60Ω
- renumbered C61 to C201, C63 to C203, JP4 to JP201, U6 to U201
Connections:
- net VCC renamed +3V3
Other:
- moved on the sheet: C203
Changed lines of the file:
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@@
+	(wire
+		(pts
+			(xy 134.62 74.93) (xy 134.62 76.2)
+		)
+		(stroke
+			(width 0)
+			(type default)
+		)
+	)
 	(wire
 		(pts
@@
 	(wire
 		(pts
+			(xy 196.85 87.63) (xy 200.66 87.63)
+		)
+		(stroke
+			(width 0)
+			(type default)
+		)
+	)
+	(wire
+		(pts
+			(xy 177.8 87.63) (xy 185.42 87.63)
+		)
+		(stroke
+			(width 0)
+			(type default)
+		)
+	)
+	(wire
+		(pts
 			(xy 134.62 76.2) (xy 137.16 76.2)
 		)
@@
 	(wire
 		(pts
-			(xy 196.85 87.63) (xy 200.66 87.63)
-		)
-		(stroke
-			(width 0)
-			(type default)
-		)
-	)
-	(wire
-		(pts
-			(xy 177.8 87.63) (xy 185.42 87.63)
-		)
-		(stroke
-			(width 0)
-			(type default)
-		)
-	)
-	(wire
-		(pts
 			(xy 177.8 95.25) (xy 177.8 96.52)
 		)
@@
 	(wire
 		(pts
+			(xy 179.07 96.52) (xy 177.8 96.52)
+		)
+		(stroke
+			(width 0)
+			(type default)
+		)
+	)
+	(wire
+		(pts
 			(xy 121.92 92.71) (xy 134.62 92.71)
 		)
@@
 	(wire
 		(pts
-			(xy 187.96 96.52) (xy 185.42 96.52)
+			(xy 187.96 96.52) (xy 186.69 96.52)
 		)
 		(stroke
@@
 	)
 	(symbol
+		(lib_id "power:+3V3")
+		(at 134.62 74.93 0)
+		(unit 1)
+		(exclude_from_sim no)
+		(in_bom yes)
+		(on_board yes)
+		(dnp no)
+		(fields_autoplaced yes)
+		(property "Reference" "#PWR0201"
+			(at 134.62 78.74 0)
+			(effects
+				(font
+					(size 1.27 1.27)
+				)
+				(hide yes)
+			)
+		)
+		(property "Value" "+3V3"
+			(at 134.62 69.85 0)
+			(effects
+				(font
+					(size 1.27 1.27)
+				)
+			)
+		)
+		(property "Footprint" ""
+			(at 134.62 74.93 0)
+			(effects
+				(font
+					(size 1.27 1.27)
+				)
+				(hide yes)
+			)
+		)
+		(property "Datasheet" ""
+			(at 134.62 74.93 0)
+			(effects
+				(font
+					(size 1.27 1.27)
+				)
+				(hide yes)
+			)
+		)
+		(property "Description" "Power symbol creates a global label with name \"+3V3\""
+			(at 134.62 74.93 0)
+			(effects
+				(font
+					(size 1.27 1.27)
+				)
+				(hide yes)
+			)
+		)
+		(pin "1"
+		)
+		(instances
+			(project "Ricardo-Garnet"
+				(path "/a4c716a5-e5f4-4cd7-812e-2c21e63f692f/00000000-0000-0000-0000-000053ffb6e1"
+					(reference "#PWR0201")
+					(unit 1)
+				)
+			)
+		)
+	)
+	(symbol
 		(lib_id "Diode:SM712_SOT23")
 		(at 196.85 96.52 270)
@@
 		(dnp no)
 		(fields_autoplaced yes)
-		(property "Reference" "D7"
-			(at 200.66 95.25 90)
+		(property "Reference" "D201"
+			(at 199.39 95.2499 90)
 			(effects
 				(font
@@
 			)
 		)
-		(property "Value" "SM712_SOT23"
-			(at 200.66 97.79 90)
+		(property "Value" "SM712"
+			(at 199.39 97.7899 90)
 			(effects
 				(font
@@
 			(project "Ricardo-Garnet"
 				(path "/a4c716a5-e5f4-4cd7-812e-2c21e63f692f/00000000-0000-0000-0000-000053ffb6e1"
-					(reference "D7")
+					(reference "D201")
 					(unit 1)
 				)
@@
 		(on_board yes)
 		(dnp no)
-		(property "Reference" "#PWR086"
+		(property "Reference" "#PWR0203"
 			(at 144.78 106.68 0)
 			(effects
@@
 			(project "Ricardo-Garnet"
 				(path "/a4c716a5-e5f4-4cd7-812e-2c21e63f692f/00000000-0000-0000-0000-000053ffb6e1"
-					(reference "#PWR086")
+					(reference "#PWR0203")
 					(unit 1)
 				)
@@
 		(on_board yes)
 		(dnp no)
-		(fields_autoplaced yes)
-		(property "Reference" "R44"
-			(at 172.72 90.17 0)
+		(property "Reference" "R202"
+			(at 174.752 83.058 0)
 			(effects
 				(font
@@
 			)
 		)
-		(property "Value" "60"
-			(at 172.72 92.71 0)
+		(property "Value" "60Ω"
+			(at 174.752 85.598 0)
 			(effects
 				(font
@@
 			(project "Ricardo-Garnet"
 				(path "/a4c716a5-e5f4-4cd7-812e-2c21e63f692f/00000000-0000-0000-0000-000053ffb6e1"
-					(reference "R44")
-					(unit 1)
-				)
-			)
-		)
-	)
-	(symbol
-		(lib_name "VCC_5")
-		(lib_id "BLDC_4-rescue:VCC")
-		(at 134.62 76.2 0)
-		(unit 1)
-		(exclude_from_sim no)
-		(in_bom yes)
-		(on_board yes)
-		(dnp no)
-		(property "Reference" "#PWR084"
-			(at 134.62 73.66 0)
-			(effects
-				(font
-					(size 0.762 0.762)
-				)
-				(hide yes)
-			)
-		)
-		(property "Value" "VCC"
-			(at 134.62 73.66 0)
-			(effects
-				(font
-					(size 0.762 0.762)
-				)
-			)
-		)
-		(property "Footprint" ""
-			(at 134.62 76.2 0)
-			(effects
-				(font
-					(size 1.524 1.524)
-				)
-				(hide yes)
-			)
-		)
-		(property "Datasheet" ""
-			(at 134.62 76.2 0)
-			(effects
-				(font
-					(size 1.524 1.524)
-				)
-				(hide yes)
-			)
-		)
-		(property "Description" ""
-			(at 134.62 76.2 0)
-			(effects
-				(font
-					(size 1.27 1.27)
-				)
-			)
-		)
-		(pin "1"
-		)
-		(instances
-			(project "Ricardo-Garnet"
-				(path "/a4c716a5-e5f4-4cd7-812e-2c21e63f692f/00000000-0000-0000-0000-000053ffb6e1"
-					(reference "#PWR084")
+					(reference "R202")
 					(unit 1)
 				)
@@
 		(dnp no)
 		(fields_autoplaced yes)
-		(property "Reference" "U6"
+		(property "Reference" "U201"
 			(at 152.4 82.7786 0)
 			(effects
@@
 			(project "Ricardo-Garnet"
 				(path "/a4c716a5-e5f4-4cd7-812e-2c21e63f692f/00000000-0000-0000-0000-000053ffb6e1"
-					(reference "U6")
+					(reference "U201")
 					(unit 1)
 				)
@@
 		(dnp no)
 		(fields_autoplaced yes)
-		(property "Reference" "C61"
+		(property "Reference" "C201"
 			(at 124.46 77.47 0)
 			(effects
@@
 			(project "Ricardo-Garnet"
 				(path "/a4c716a5-e5f4-4cd7-812e-2c21e63f692f/00000000-0000-0000-0000-000053ffb6e1"
-					(reference "C61")
+					(reference "C201")
 					(unit 1)
 				)
@@
 		(dnp no)
 		(fields_autoplaced yes)
-		(property "Reference" "JP4"
+		(property "Reference" "JP201"
 			(at 167.64 90.17 0)
 			(effects
@@
 			(project "Ricardo-Garnet"
 				(path "/a4c716a5-e5f4-4cd7-812e-2c21e63f692f/00000000-0000-0000-0000-000053ffb6e1"
-					(reference "JP4")
+					(reference "JP201")
 					(unit 1)
 				)
@@
 		(dnp no)
 		(fields_autoplaced yes)
-		(property "Reference" "C62"
+		(property "Reference" "C202"
 			(at 139.7 77.4762 0)
 			(effects
@@
 			)
 		)
-		(property "Footprint" "Capacitor_SMD:C_0402_1005Metric"
+		(property "Footprint" "Capacitor_SMD:C_0603_1608Metric"
 			(at 137.16 78.74 0)
 			(effects
@@
 			(project "Ricardo-Garnet"
 				(path "/a4c716a5-e5f4-4cd7-812e-2c21e63f692f/00000000-0000-0000-0000-000053ffb6e1"
-					(reference "C62")
+					(reference "C202")
 					(unit 1)
 				)
@@
 		(on_board yes)
 		(dnp no)
-		(property "Reference" "#PWR085"
+		(property "Reference" "#PWR0202"
 			(at 134.62 82.55 0)
 			(effects
@@
 			(project "Ricardo-Garnet"
 				(path "/a4c716a5-e5f4-4cd7-812e-2c21e63f692f/00000000-0000-0000-0000-000053ffb6e1"
-					(reference "#PWR085")
+					(reference "#PWR0202")
 					(unit 1)
 				)
@@
 	(symbol
 		(lib_id "Device:C")
-		(at 181.61 96.52 90)
+		(at 182.88 96.52 90)
 		(unit 1)
 		(exclude_from_sim no)
@@
 		(dnp no)
 		(fields_autoplaced yes)
-		(property "Reference" "C63"
-			(at 181.61 90.17 90)
+		(property "Reference" "C203"
+			(at 182.88 90.17 90)
 			(effects
 				(font
@@
 		)
 		(property "Value" "47nF"
-			(at 181.61 92.71 90)
+			(at 182.88 92.71 90)
 			(effects
 				(font
@@
 		)
 		(property "Footprint" "Capacitor_SMD:C_0402_1005Metric"
-			(at 185.42 95.5548 0)
+			(at 186.69 95.5548 0)
 			(effects
 				(font
@@
 		)
 		(property "Datasheet" "~"
-			(at 181.61 96.52 0)
+			(at 182.88 96.52 0)
 			(effects
 				(font
@@
 		)
 		(property "Description" "Unpolarized capacitor"
-			(at 181.61 96.52 0)
+			(at 182.88 96.52 0)
 			(effects
 				(font
@@
 			(project "Ricardo-Garnet"
 				(path "/a4c716a5-e5f4-4cd7-812e-2c21e63f692f/00000000-0000-0000-0000-000053ffb6e1"
-					(reference "C63")
+					(reference "C203")
 					(unit 1)
 				)
@@
 		(dnp no)
 		(fields_autoplaced yes)
-		(property "Reference" "#PWR087"
+		(property "Reference" "#PWR0204"
 			(at 187.96 102.87 0)
 			(effects
@@
 			(project "Ricardo-Garnet"
 				(path "/a4c716a5-e5f4-4cd7-812e-2c21e63f692f/00000000-0000-0000-0000-000053ffb6e1"
-					(reference "#PWR087")
+					(reference "#PWR0204")
 					(unit 1)
 				)
@@
 		(on_board yes)
 		(dnp no)
-		(property "Reference" "R41"
+		(property "Reference" "R201"
 			(at 128.27 101.6 0)
 			(effects
@@
 			)
 		)
-		(property "Value" "0"
+		(property "Value" "0Ω"
 			(at 128.27 104.14 0)
 			(effects
@@
 			(project "Ricardo-Garnet"
 				(path "/a4c716a5-e5f4-4cd7-812e-2c21e63f692f/00000000-0000-0000-0000-000053ffb6e1"
-					(reference "R41")
+					(reference "R201")
 					(unit 1)
 				)
@@
 		(on_board yes)
 		(dnp no)
-		(fields_autoplaced yes)
-		(property "Reference" "R45"
-			(at 172.72 100.33 0)
+		(property "Reference" "R203"
+			(at 175.26 107.442 0)
 			(effects
 				(font
@@
 			)
 		)
-		(property "Value" "60"
-			(at 172.72 102.87 0)
+		(property "Value" "60Ω"
+			(at 175.26 109.982 0)
 			(effects
 				(font
@@
 			(project "Ricardo-Garnet"
 				(path "/a4c716a5-e5f4-4cd7-812e-2c21e63f692f/00000000-0000-0000-0000-000053ffb6e1"
-					(reference "R45")
-					(unit 1)
-				)
+					(reference "R203")
+					(unit 1)
+				)
