File: Hardware/boosts_sch.kicad_sch (KiCad schematic)
At the start: 47 parts, among them IC1 TPS61089RNRR, IC2 AP2205-W5-7, IC3 AP2205-W5-7, IC4 TPS61089RNRR, U8 SMA6J5.0A

Commit message: removed voltage pt sensing capabilities
Parts:
- removed C48: 10uF, Capacitor_SMD:C_0603_1608Metric, symbol Device:C_Small
- removed C50: 180pF, Capacitor_SMD:C_0402_1005Metric, symbol Device:C_Small
- removed C53: 3.9nF, Capacitor_SMD:C_0402_1005Metric, symbol Device:C_Small
- removed C54: 1uF, Capacitor_SMD:C_0402_1005Metric, symbol Device:C_Small
- removed C55, C56: 22uF, Capacitor_SMD:C_0805_2012Metric, symbol Device:C_Small
- removed C57, C59, C65: 100nF, Capacitor_SMD:C_0402_1005Metric, symbol Device:C_Small
- removed C58: 2.2uF, Capacitor_SMD:C_0402_1005Metric, symbol Device:C_Small
- removed C60: 47uF, Capacitor_SMD:C_1206_3216Metric, symbol Device:C_Small
- removed C64: 10uF, Capacitor_SMD:C_0402_1005Metric, symbol Device:C_Small
- removed IC1: TPS61089RNRR, iclr:IC_TPS61089RNRR, symbol iclr:TPS61089RNRR
- removed IC2: AP2205-W5-7, iclr:SOT95P282X145-5N, symbol iclr:AP2205-W5-7
- removed L2: SRR6038-5R0Y, iclr:IND_SRP6540-390M, symbol iclr:SRR6038-5R0Y
- removed R12: 7.87k, Resistor_SMD:R_0402_1005Metric, symbol Device:R_Small
- removed R13: 360k, Resistor_SMD:R_0402_1005Metric, symbol Device:R_Small
- removed R22: 49.9k, Resistor_SMD:R_0402_1005Metric, symbol Device:R_Small
- removed R22: 100k, Resistor_SMD:R_0402_1005Metric, symbol Device:R_Small
- removed R37: 10K, Resistor_SMD:R_0402_1005Metric, symbol Device:R_Small
- removed R38: 562k, Resistor_SMD:R_0402_1005Metric, symbol Device:R_Small
- removed R47: 150k, Resistor_SMD:R_0402_1005Metric, symbol Device:R_Small
- removed R52: 301k, Resistor_SMD:R_0402_1005Metric, symbol Device:R_Small
- removed U8: SMA6J5.0A, symbol ICLR_HW:SMA6J5.0A
Other:
- note removed: "BOOST"
- note removed: "LDO"
- note removed: "SIM: https://webench.ti.com/appinfo/webench/scripts/SDP.cgi?ID=C25BB1AA15C31C1A"
- moved on the sheet: C75, C76

Commit message: changes made post will's review
Parts:
- removed C66: 1uF, Capacitor_SMD:C_0402_1005Metric, symbol Device:C_Small
- removed C70, C72: 10uF, Capacitor_SMD:C_0805_2012Metric, symbol Device:C_Small
- removed C71: 2.2uF, Capacitor_SMD:C_0402_1005Metric, symbol Device:C_Small
- removed C75: 10uF, Capacitor_SMD:C_0603_1608Metric, symbol Device:C_Small
- removed C76: 100nF, Capacitor_SMD:C_0402_1005Metric, symbol Device:C_Small
- added C407, C411: 100nF, Capacitor_SMD:C_0402_1005Metric, symbol Device:C_Small
- added C408, C409: 10uF, Capacitor_SMD:C_0805_2012Metric, symbol Device:C_Small
- added C410: 1uF, Capacitor_SMD:C_0603_1608Metric, symbol Device:C_Small
- R401: renamed from R57; value 28.7k -> 28.7kΩ
- R402: renamed from R58; value 866k -> 866kΩ
- R403: renamed from R59; value 92k -> 92kΩ
- R404: renamed from R61; value 10K -> 10kΩ
- R405: renamed from R62; value 332k -> 332kΩ
- R406: renamed from R63; value 280k -> 280kΩ
- R407: renamed from R60; value 49.9k -> 49.9kΩ
- R408: renamed from R65; value 432k -> 432kΩ
- renumbered C67 to C401, C68 to C402, C69 to C403, C73 to C404, C74 to C405, C48 to C406, IC4 to IC401, IC3 to IC402, L6 to L401
Connections:
- net 12V: now also C410.1, C411.1
- net GND: now also C407.2, C408.2, C409.2, C410.2, C411.2
- net LDO12.6V_IN: now also C407.1, C408.1, C409.1
- net VCC renamed +3V3
Other:
- moved on the sheet: C401, C402, C403, C404, C405, C406, IC401, IC402, L401, R401, R402, R403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
