File: Hardware/power.kicad_sch (KiCad schematic)
At the start: 18 parts, among them U4 LM66200DRLR, U4 MAX77827AEFD+T, U5 SC4215

Commit message: chatting to fang
Parts:
- renumbered U4 to U7
Changed lines of the file:
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@@
 		(dnp no)
 		(fields_autoplaced yes)
-		(property "Reference" "U4"
+		(property "Reference" "U7"
 			(at 149.86 69.9602 0)
 			(effects
@@
 			(project "BLDC_4"
 				(path "/a4c716a5-e5f4-4cd7-812e-2c21e63f692f/6f1e0e7e-af26-435a-9a05-4d550e4eb21c"
-					(reference "U4")
+					(reference "U7")
 					(unit 1)
 				)

Commit message: changes made post will's review
Parts:
- removed C3: 10uF, Capacitor_SMD:C_0402_1005Metric, symbol Device:C_Small
- removed C38: 22uF, Capacitor_SMD:C_0603_1608Metric, symbol Device:C_Small
- removed C45: 4.7uF, Capacitor_SMD:C_0402_1005Metric, symbol Device:C_Small
- added C303, C305, C306: 10uF, Capacitor_SMD:C_0603_1608Metric, symbol Device:C_Small
- C304: renamed from C42; footprint Capacitor_SMD:C_0402_1005Metric -> Capacitor_SMD:C_0603_1608Metric
- C308: renamed from C47; value 0.1uF -> 100nF
- R301: renamed from R14; value 10k -> 10kΩ
- R302: renamed from R15; value 14k -> 14kΩ
- R303: renamed from R16; value 56k -> 56kΩ
- R304: renamed from R11; value 10k -> 10kΩ
- renumbered C32 to C301, C35 to C302, C46 to C307, L3 to L301, TP5 to TP301, TP6 to TP302, U4 to U301, U7 to U302, U5 to U303
Connections:
- net BBOUT: now also C303.1, C305.1, C306.1
- net GND: now also C303.2, C305.2, C306.2
- net VCC renamed +3V3
Other:
- moved on the sheet: C307, C308, TP301, TP302
