File: Hardware/usb.kicad_sch (KiCad schematic)
At the start: 8 parts, among them J2 USB_C_Receptacle_USB2.0

Commit message: changes made post will's review
Parts:
- removed TP1, TP2: TestPoint, TestPoint:TestPoint_Pad_D1.0mm, symbol Connector:TestPoint
- R801: renamed from R31; value 5.1k -> 5.1kΩ
- R802: renamed from R39; value 5.1k -> 5.1kΩ
- R803: renamed from R40; value 5.1k -> 5.1kΩ
- renumbered D6 to D801, J2 to J801, LED6 to LED801
Connections:
- net +5V: now also D801.4 (K); no longer D801.2 (K)
- net Data+: now also D801.3 (K); no longer D801.4 (K)
- net Data-: now also D801.2 (K); no longer D801.3 (K)
